File: mini_fpga_control.sch (KiCad schematic (older format))
At the start: 10 parts

Commit message: Complete control/storage section (hopefully!)
Parts:
- added C?: .01u, ~, symbol C
- added J?: JTAG_1X6, symbol JTAG_1X6
- added J?: USD_SLOT, symbol USD_SLOT
- added U?: CPPC7, symbol CPPC7
Connections:
- wire segments 48 -> 87
Changed lines of the file:
@@
 	8250 6400 8150 6400
 Connection ~ 8250 6000
+$Comp
+L JTAG_1X6 J?
+U 1 1 53D083B5
+P 5800 1550
+F 0 "J?" H 5650 1150 60  0000 C CNN
+F 1 "JTAG_1X6" H 5800 1950 60  0000 C CNN
+F 2 "" H 5800 1550 60  0000 C CNN
+F 3 "" H 5800 1550 60  0000 C CNN
+	1    5800 1550
+	1    0    0    -1
+$EndComp
+Wire Wire Line
+	5300 1300 4150 1300
+Wire Wire Line
+	5300 1400 4150 1400
+Wire Wire Line
+	5300 1500 4150 1500
+Wire Wire Line
+	5300 1600 4150 1600
+Wire Wire Line
+	5300 1800 5200 1800
+Wire Wire Line
+	5200 1800 5200 1900
+$Comp
+L GND #PWR?
+U 1 1 53D08593
+P 5200 1900
+F 0 "#PWR?" H 5200 1900 30  0001 C CNN
+F 1 "GND" H 5200 1830 30  0001 C CNN
+F 2 "" H 5200 1900 60  0000 C CNN
+F 3 "" H 5200 1900 60  0000 C CNN
+	1    5200 1900
+	1    0    0    -1
+$EndComp
+$Comp
+L +3.3V #PWR?
+U 1 1 53D085A0
+P 4950 1700
+F 0 "#PWR?" H 4950 1660 30  0001 C CNN
+F 1 "+3.3V" H 4950 1810 30  0000 C CNN
+F 2 "" H 4950 1700 60  0000 C CNN
+F 3 "" H 4950 1700 60  0000 C CNN
+	1    4950 1700
+	1    0    0    -1
+$EndComp
+Wire Wire Line
+	5300 1700 4950 1700
+$Comp
+L USD_SLOT J?
+U 1 1 53D0874F
+P 9300 4950
+F 0 "J?" H 9200 4400 60  0000 C CNN
+F 1 "USD_SLOT" H 9350 5300 60  0000 C CNN
+F 2 "" H 9300 4950 60  0000 C CNN
+F 3 "" H 9300 4950 60  0000 C CNN
+	1    9300 4950
+	1    0    0    -1
+$EndComp
+Wire Wire Line
+	7100 4500 8550 4500
+Wire Wire Line
+	8550 4500 8550 4700
+Wire Wire Line
+	8550 4700 8850 4700
+Wire Wire Line
+	7100 4600 8450 4600
+Wire Wire Line
+	8450 4600 8450 4800
+Wire Wire Line
+	8450 4800 8850 4800
+Wire Wire Line
+	7100 4800 8350 4800
+Wire Wire Line
+	8350 4800 8350 4900
+Wire Wire Line
+	8350 4900 8850 4900
+Wire Wire Line
+	7100 4900 8250 4900
+Wire Wire Line
+	8250 4900 8250 5100
+Wire Wire Line
+	8250 5100 8850 5100
+Wire Wire Line
+	7100 5100 8150 5100
+Wire Wire Line
+	8150 5100 8150 5300
+Wire Wire Line
+	8150 5300 8850 5300
+Wire Wire Line
+	7100 5200 8050 5200
+Wire Wire Line
+	8050 5200 8050 5400
+Wire Wire Line
+	8050 5400 8850 5400
+Wire Wire Line
+	8850 5000 8750 5000
+Wire Wire Line
+	8750 5000 8750 4350
+Wire Wire Line
+	8850 5200 8750 5200
+Wire Wire Line
+	8750 5200 8750 5650
+$Comp
+L +3.3V #PWR?
+U 1 1 53D08A4E
+P 8750 4350
+F 0 "#PWR?" H 8750 4310 30  0001 C CNN
+F 1 "+3.3V" H 8750 4460 30  0000 C CNN
+F 2 "" H 8750 4350 60  0000 C CNN
+F 3 "" H 8750 4350 60  0000 C CNN
+	1    8750 4350
+	1    0    0    -1
+$EndComp
+$Comp
+L GND #PWR?
+U 1 1 53D08A56
+P 8750 5650
+F 0 "#PWR?" H 8750 5650 30  0001 C CNN
+F 1 "GND" H 8750 5580 30  0001 C CNN
+F 2 "" H 8750 5650 60  0000 C CNN
+F 3 "" H 8750 5650 60  0000 C CNN
+	1    8750 5650
+	1    0    0    -1
+$EndComp
+$Comp
+L CPPC7 U?
+U 1 1 53D08BD0
+P 8000 2850
+F 0 "U?" H 7750 3000 60  0000 C CNN
+F 1 "CPPC7" H 8150 3000 60  0000 C CNN
+F 2 "" H 7900 2850 60  0000 C CNN
+F 3 "" H 7900 2850 60  0000 C CNN
+	1    8000 2850
+	1    0    0    -1
+$EndComp
+Wire Wire Line
+	8600 2900 8600 3300
+Wire Wire Line
+	8600 3300 7100 3300
+Wire Wire Line
+	7400 2100 7400 2800
+Wire Wire Line
+	6750 2100 8600 2100
+$Comp
+L +3.3V #PWR?
+U 1 1 53D08C89
+P 6750 2050
+F 0 "#PWR?" H 6750 2010 30  0001 C CNN
+F 1 "+3.3V" H 6750 2160 30  0000 C CNN
+F 2 "" H 6750 2050 60  0000 C CNN
+F 3 "" H 6750 2050 60  0000 C CNN
+	1    6750 2050
+	1    0    0    -1
+$EndComp
+Wire Wire Line
+	6750 2100 6750 2050
+Wire Wire Line
+	8600 2100 8600 2800
+Connection ~ 7400 2100
+$Comp
+L GND #PWR?
+U 1 1 53D08D40
+P 6750 2950
+F 0 "#PWR?" H 6750 2950 30  0001 C CNN
+F 1 "GND" H 6750 2880 30  0001 C CNN
+F 2 "" H 6750 2950 60  0000 C CNN
+F 3 "" H 6750 2950 60  0000 C CNN
+	1    6750 2950
+	1    0    0    -1
+$EndComp
+Wire Wire Line
+	7400 2900 6750 2900
+Wire Wire Line
+	6750 2900 6750 2950
+$Comp
+L C C?
+U 1 1 53D08DA3
+P 7000 2500
+F 0 "C?" H 7000 2600 40  0000 L CNN
+F 1 ".01u" H 7006 2415 40  0000 L CNN
+F 2 "~" H 7038 2350 30  0000 C CNN
+F 3 "~" H 7000 2500 60  0000 C CNN
+	1    7000 2500
+	1    0    0    -1
+$EndComp
+Wire Wire Line
+	7000 2100 7000 2300
+Connection ~ 7000 2100
+Wire Wire Line
+	7000 2700 7000 2900
+Connection ~ 7000 2900
 $EndSCHEMATC

Commit message: First checkover of schematic complete, should be working.
Parts:
- added R?: 4.7K, ~, symbol R
Connections:
- wire segments 87 -> 89
- no-connect marks 1 -> 25
Other:
- note added: "Do not populate"
Changed lines of the file:
@@
 Sheet 5 6
 Title ""
-Date "26 jul 2014"
+Date "28 jul 2014"
 Rev ""
 Comp ""
@@
 $EndComp
 Wire Wire Line
-	5700 6500 5900 6500
+	5500 6500 5900 6500
 Wire Wire Line
 	6400 6500 6550 6500
@@
 	7000 2700 7000 2900
 Connection ~ 7000 2900
+NoConn ~ 4300 3900
+NoConn ~ 4300 4000
+NoConn ~ 4300 4500
+NoConn ~ 4300 4600
+NoConn ~ 4300 4900
+NoConn ~ 4300 5100
+NoConn ~ 4300 5200
+NoConn ~ 4300 5400
+NoConn ~ 4300 5500
+NoConn ~ 4300 5700
+NoConn ~ 4300 5800
+NoConn ~ 4300 6000
+NoConn ~ 4300 6100
+NoConn ~ 7100 5800
+NoConn ~ 7100 5700
+NoConn ~ 7100 5500
+NoConn ~ 7100 5400
+NoConn ~ 7100 4300
+NoConn ~ 7100 4200
+NoConn ~ 7100 4000
+NoConn ~ 7100 3900
+NoConn ~ 7100 3700
+NoConn ~ 7100 3600
+NoConn ~ 7100 3400
+$Comp
+L R R?
+U 1 1 53D58328
+P 5250 6500
+F 0 "R?" V 5330 6500 40  0000 C CNN
+F 1 "4.7K" V 5257 6501 40  0000 C CNN
+F 2 "~" V 5180 6500 30  0000 C CNN
+F 3 "~" H 5250 6500 30  0000 C CNN
+	1    5250 6500
+	0    -1   -1   0
+$EndComp
+Connection ~ 5700 6500
+$Comp
+L GND #PWR?
+U 1 1 53D5838F
+P 4900 6600
+F 0 "#PWR?" H 4900 6600 30  0001 C CNN
+F 1 "GND" H 4900 6530 30  0001 C CNN
+F 2 "" H 4900 6600 60  0000 C CNN
+F 3 "" H 4900 6600 60  0000 C CNN
+	1    4900 6600
+	1    0    0    -1
+$EndComp
+Wire Wire Line
+	5000 6500 4900 6500
+Wire Wire Line
+	4900 6500 4900 6600
+Text Notes 4700 6400 0    60   ~ 0
+Do not populate
 $EndSCHEMATC

Commit message: Annotated!
Parts:
- gave numbers to parts that had none: 14
Changed lines of the file:
@@
 $EndDescr
 $Comp
-L XC6SLX9 U?
+L XC6SLX9 U3
 U 2 1 53CA8289
 P 3450 1550
-F 0 "U?" H 3450 1450 60  0000 C CNN
+F 0 "U3" H 3450 1450 60  0000 C CNN
 F 1 "XC6SLX9" H 3450 1650 60  0000 C CNN
 F 2 "~" H 3600 3550 60  0000 C CNN
@@
 $EndComp
 $Comp
-L XC6SLX9 U?
+L XC6SLX9 U3
 U 5 1 53C9F822
 P 5700 4550
-F 0 "U?" H 5700 4450 60  0000 C CNN
+F 0 "U3" H 5700 4450 60  0000 C CNN
 F 1 "XC6SLX9" H 5700 4650 60  0000 C CNN
 F 2 "~" H 5850 6550 60  0000 C CNN
@@
 $EndComp
 $Comp
-L GND #PWR05
+L GND #PWR45
 U 1 1 53C9F88B
 P 4150 5000
-F 0 "#PWR05" H 4150 5000 30  0001 C CNN
+F 0 "#PWR45" H 4150 5000 30  0001 C CNN
 F 1 "GND" H 4150 4930 30  0001 C CNN
 F 2 "" H 4150 5000 60  0000 C CNN
@@
 	4150 4800 4150 5000
 $Comp
-L S25FL164 U?
+L S25FL164 U5
 U 1 1 53C9FB3A
 P 2200 4550
-F 0 "U?" H 2200 4650 60  0000 C CNN
+F 0 "U5" H 2200 4650 60  0000 C CNN
 F 1 "S25FL164" H 2200 4450 60  0000 C CNN
 F 2 "~" H 2200 4550 60  0000 C CNN
@@
 $EndComp
 $Comp
-L +3.3V #PWR07
+L +3.3V #PWR44
 U 1 1 53C9FB73
 P 3350 4150
-F 0 "#PWR07" H 3350 4110 30  0001 C CNN
+F 0 "#PWR44" H 3350 4110 30  0001 C CNN
 F 1 "+3.3V" H 3350 4260 30  0000 C CNN
 F 2 "" H 3350 4150 60  0000 C CNN
@@
 $EndComp
 $Comp
-L GND #PWR08
+L GND #PWR41
 U 1 1 53C9FB79
 P 1100 5000
-F 0 "#PWR08" H 1100 5000 30  0001 C CNN
+F 0 "#PWR41" H 1100 5000 30  0001 C CNN
 F 1 "GND" H 1100 4930 30  0001 C CNN
 F 2 "" H 1100 5000 60  0000 C CNN
@@
 	3550 4650 3200 4650
 $Comp
-L +3.3V #PWR09
+L +3.3V #PWR40
 U 1 1 53C9FD59
 P 600 4550
-F 0 "#PWR09" H 600 4510 30  0001 C CNN
+F 0 "#PWR40" H 600 4510 30  0001 C CNN
 F 1 "+3.3V" H 600 4660 30  0000 C CNN
 F 2 "" H 600 4550 60  0000 C CNN
@@
 Connection ~ 3350 4250
 $Comp
-L R R?
+L R R48
 U 1 1 53CAE7AD
 P 6150 6500
-F 0 "R?" V 6230 6500 40  0000 C CNN
+F 0 "R48" V 6230 6500 40  0000 C CNN
 F 1 "4.7K" V 6157 6501 40  0000 C CNN
 F 2 "~" V 6080 6500 30  0000 C CNN
@@
 $EndComp
 $Comp
-L +3.3V #PWR010
+L +3.3V #PWR50
 U 1 1 53CAE7BA
 P 6550 6400
-F 0 "#PWR010" H 6550 6360 30  0001 C CNN
+F 0 "#PWR50" H 6550 6360 30  0001 C CNN
 F 1 "+3.3V" H 6550 6510 30  0000 C CNN
 F 2 "" H 6550 6400 60  0000 C CNN
@@
 	6550 6500 6550 6400
 $Comp
-L R R?
+L R R49
 U 1 1 53CAE986
 P 7900 6000
-F 0 "R?" V 7980 6000 40  0000 C CNN
+F 0 "R49" V 7980 6000 40  0000 C CNN
 F 1 "4.7K" V 7907 6001 40  0000 C CNN
 F 2 "~" V 7830 6000 30  0000 C CNN
@@
 $EndComp
 $Comp
-L +3.3V #PWR011
+L +3.3V #PWR53
 U 1 1 53CAE9AC
 P 8250 5900
-F 0 "#PWR011" H 8250 5860 30  0001 C CNN
+F 0 "#PWR53" H 8250 5860 30  0001 C CNN
 F 1 "+3.3V" H 8250 6010 30  0000 C CNN
 F 2 "" H 8250 5900 60  0000 C CNN
@@
 	1100 4450 1200 4450
 $Comp
-L R R?
+L R R43
 U 1 1 53CAED90
 P 2150 4000
-F 0 "R?" V 2230 4000 40  0000 C CNN
+F 0 "R43" V 2230 4000 40  0000 C CNN
 F 1 "100" V 2157 4001 40  0000 C CNN
 F 2 "~" V 2080 4000 30  0000 C CNN
@@
 	1900 4000 1100 4000
 $Comp
-L GND #PWR?
+L GND #PWR46
 U 1 1 53CAEFE3
 P 4250 1950
-F 0 "#PWR?" H 4250 1950 30  0001 C CNN
+F 0 "#PWR46" H 4250 1950 30  0001 C CNN
 F 1 "GND" H 4250 1880 30  0001 C CNN
 F 2 "" H 4250 1950 60  0000 C CNN
@@
 	4250 1850 4250 1950
 $Comp
-L R R?
+L R R46
 U 1 1 53CAF070
 P 3550 3250
-F 0 "R?" V 3630 3250 40  0000 C CNN
+F 0 "R46" V 3630 3250 40  0000 C CNN
 F 1 "330" V 3557 3251 40  0000 C CNN
 F 2 "~" V 3480 3250 30  0000 C CNN
@@
 $EndComp
 $Comp
-L +3.3V #PWR?
+L +3.3V #PWR43
 U 1 1 53CAF07D
 P 3100 3100
-F 0 "#PWR?" H 3100 3060 30  0001 C CNN
+F 0 "#PWR43" H 3100 3060 30  0001 C CNN
 F 1 "+3.3V" H 3100 3210 30  0000 C CNN
 F 2 "" H 3100 3100 60  0000 C CNN
@@
 Connection ~ 3100 3250
 $Comp
-L R R?
+L R R44
 U 1 1 53CAF101
 P 2250 2950
-F 0 "R?" V 2330 2950 40  0000 C CNN
+F 0 "R44" V 2330 2950 40  0000 C CNN
 F 1 "100" V 2257 2951 40  0000 C CNN
 F 2 "~" V 2180 2950 30  0000 C CNN
@@
 $EndComp
 $Comp
-L R R?
+L R R45
 U 1 1 53CAF120
 P 2250 3550
-F 0 "R?" V 2330 3550 40  0000 C CNN
+F 0 "R45" V 2330 3550 40  0000 C CNN
 F 1 "100" V 2257 3551 40  0000 C CNN
 F 2 "~" V 2180 3550 30  0000 C CNN
@@
 Connection ~ 2250 3250
 $Comp
-L GND #PWR?
+L GND #PWR42
 U 1 1 53CAF1E3
 P 2250 3850
-F 0 "#PWR?" H 2250 3850 30  0001 C CNN
+F 0 "#PWR42" H 2250 3850 30  0001 C CNN
 F 1 "GND" H 2250 3780 30  0001 C CNN
 F 2 "" H 2250 3850 60  0000 C CNN
@@
 Connection ~ 7350 6100
 $Comp
-L R R?
+L R R50
 U 1 1 53CAF24E
 P 7900 6400
-F 0 "R?" V 7980 6400 40  0000 C CNN
+F 0 "R50" V 7980 6400 40  0000 C CNN
 F 1 "4.7K" V 7907 6401 40  0000 C CNN
 F 2 "~" V 7830 6400 30  0000 C CNN
@@
 Connection ~ 8250 6000
 $Comp
-L JTAG_1X6 J?
+L JTAG_1X6 J4
 U 1 1 53D083B5
 P 5800 1550
-F 0 "J?" H 5650 1150 60  0000 C CNN
+F 0 "J4" H 5650 1150 60  0000 C CNN
 F 1 "JTAG_1X6" H 5800 1950 60  0000 C CNN
 F 2 "" H 5800 1550 60  0000 C CNN
@@
 	5200 1800 5200 1900
 $Comp
-L GND #PWR?
+L GND #PWR49
 U 1 1 53D08593
 P 5200 1900
-F 0 "#PWR?" H 5200 1900 30  0001 C CNN
+F 0 "#PWR49" H 5200 1900 30  0001 C CNN
 F 1 "GND" H 5200 1830 30  0001 C CNN
 F 2 "" H 5200 1900 60  0000 C CNN
@@
 $EndComp
 $Comp
-L +3.3V #PWR?
+L +3.3V #PWR48
 U 1 1 53D085A0
 P 4950 1700
-F 0 "#PWR?" H 4950 1660 30  0001 C CNN
+F 0 "#PWR48" H 4950 1660 30  0001 C CNN
 F 1 "+3.3V" H 4950 1810 30  0000 C CNN
 F 2 "" H 4950 1700 60  0000 C CNN
@@
 	5300 1700 4950 1700
 $Comp
-L USD_SLOT J?
+L USD_SLOT J5
 U 1 1 53D0874F
 P 9300 4950
-F 0 "J?" H 9200 4400 60  0000 C CNN
+F 0 "J5" H 9200 4400 60  0000 C CNN
 F 1 "USD_SLOT" H 9350 5300 60  0000 C CNN
 F 2 "" H 9300 4950 60  0000 C CNN
@@
 	8750 5200 8750 5650
 $Comp
-L +3.3V #PWR?
+L +3.3V #PWR54
 U 1 1 53D08A4E
 P 8750 4350
-F 0 "#PWR?" H 8750 4310 30  0001 C CNN
+F 0 "#PWR54" H 8750 4310 30  0001 C CNN
 F 1 "+3.3V" H 8750 4460 30  0000 C CNN
 F 2 "" H 8750 4350 60  0000 C CNN
@@
 $EndComp
 $Comp
-L GND #PWR?
+L GND #PWR55
 U 1 1 53D08A56
 P 8750 5650
-F 0 "#PWR?" H 8750 5650 30  0001 C CNN
+F 0 "#PWR55" H 8750 5650 30  0001 C CNN
 F 1 "GND" H 8750 5580 30  0001 C CNN
 F 2 "" H 8750 5650 60  0000 C CNN
@@
 $EndComp
 $Comp
-L CPPC7 U?
+L CPPC7 U6
 U 1 1 53D08BD0
 P 8000 2850
-F 0 "U?" H 7750 3000 60  0000 C CNN
+F 0 "U6" H 7750 3000 60  0000 C CNN
 F 1 "CPPC7" H 8150 3000 60  0000 C CNN
 F 2 "" H 7900 2850 60  0000 C CNN
@@
 	6750 2100 8600 2100
 $Comp
-L +3.3V #PWR?
+L +3.3V #PWR51
 U 1 1 53D08C89
 P 6750 2050
-F 0 "#PWR?" H 6750 2010 30  0001 C CNN
+F 0 "#PWR51" H 6750 2010 30  0001 C CNN
 F 1 "+3.3V" H 6750 2160 30  0000 C CNN
 F 2 "" H 6750 2050 60  0000 C CNN
@@
 Connection ~ 7400 2100
 $Comp
-L GND #PWR?
+L GND #PWR52
 U 1 1 53D08D40
 P 6750 2950
-F 0 "#PWR?" H 6750 2950 30  0001 C CNN
+F 0 "#PWR52" H 6750 2950 30  0001 C CNN
 F 1 "GND" H 6750 2880 30  0001 C CNN
 F 2 "" H 6750 2950 60  0000 C CNN
@@
 	6750 2900 6750 2950
 $Comp
-L C C?
+L C C48
 U 1 1 53D08DA3
 P 7000 2500
-F 0 "C?" H 7000 2600 40  0000 L CNN
+F 0 "C48" H 7000 2600 40  0000 L CNN
 F 1 ".01u" H 7006 2415 40  0000 L CNN
 F 2 "~" H 7038 2350 30  0000 C CNN
@@
 NoConn ~ 7100 3400
 $Comp
-L R R?
+L R R47
 U 1 1 53D58328
 P 5250 6500
-F 0 "R?" V 5330 6500 40  0000 C CNN
+F 0 "R47" V 5330 6500 40  0000 C CNN
 F 1 "4.7K" V 5257 6501 40  0000 C CNN
 F 2 "~" V 5180 6500 30  0000 C CNN
@@
 Connection ~ 5700 6500
 $Comp
-L GND #PWR?
+L GND #PWR47
 U 1 1 53D5838F
 P 4900 6600
-F 0 "#PWR?" H 4900 6600 30  0001 C CNN
+F 0 "#PWR47" H 4900 6600 30  0001 C CNN
 F 1 "GND" H 4900 6530 30  0001 C CNN
 F 2 "" H 4900 6600 60  0000 C CNN

Commit message: minor edits to components to fix some pin assignment issues.
Parts:
- added C49, C50: 100n, ~, symbol C
Connections:
- wire segments 89 -> 97
Changed lines of the file:
@@
 	3350 4250 3200 4250
 Wire Wire Line
-	1200 4850 1100 4850
+	900  4850 1200 4850
 Wire Wire Line
 	1100 4850 1100 5000
@@
 	600  4550 600  4650
 Wire Wire Line
-	3350 4150 3350 4450
+	3350 4150 3350 5050
 Wire Wire Line
 	3350 4450 3200 4450
@@
 Text Notes 4700 6400 0    60   ~ 0
 Do not populate
+$Comp
+L C C49
+U 1 1 53D6D42F
+P 3350 5250
+F 0 "C49" H 3350 5350 40  0000 L CNN
+F 1 "100n" H 3356 5165 40  0000 L CNN
+F 2 "~" H 3388 5100 30  0000 C CNN
+F 3 "~" H 3350 5250 60  0000 C CNN
+	1    3350 5250
+	1    0    0    -1
+$EndComp
+Connection ~ 3350 4450
+Wire Wire Line
+	3350 5450 900  5450
+Wire Wire Line
+	900  5450 900  4850
+Connection ~ 1100 4850
+$Comp
+L C C50
+U 1 1 53D6D51C
+P 8200 4150
+F 0 "C50" H 8200 4250 40  0000 L CNN
+F 1 "100n" H 8206 4065 40  0000 L CNN
+F 2 "~" H 8238 4000 30  0000 C CNN
+F 3 "~" H 8200 4150 60  0000 C CNN
+	1    8200 4150
+	1    0    0    -1
+$EndComp
+Wire Wire Line
+	8200 3950 8650 3950
+Wire Wire Line
+	8650 3950 8650 4500
+Wire Wire Line
+	8650 4500 8750 4500
+Connection ~ 8750 4500
+Wire Wire Line
+	8200 4350 7950 4350
+Wire Wire Line
+	7950 4350 7950 5550
+Wire Wire Line
+	7950 5550 8750 5550
+Connection ~ 8750 5550
 $EndSCHEMATC
