File: mini_fpga_io.sch (KiCad schematic (older format))
At the start: 17 parts, among them J2 1X6_HEADER, J3 1X6_HEADER, U3 XC6SLX9

Commit message: Almost completed all footprints.
Connections:
- net GND: now also J3.5 (GND)
Changed lines of the file:
@@
 Sheet 4 6
 Title ""
-Date "29 jul 2014"
+Date "30 jul 2014"
 Rev ""
 Comp ""
@@
 	9900 2500 9800 2500
 $Comp
-L +3.3V #PWR038
+L +3.3V #PWR037
 U 1 1 53D59B4F
 P 10250 3100
-F 0 "#PWR038" H 10250 3060 30  0001 C CNN
+F 0 "#PWR037" H 10250 3060 30  0001 C CNN
 F 1 "+3.3V" H 10250 3210 30  0000 C CNN
 F 2 "" H 10250 3100 60  0000 C CNN
@@
 Connection ~ 9800 3200
 $Comp
-L GND #PWR039
+L GND #PWR038
 U 1 1 53D59B8D
 P 9750 4450
-F 0 "#PWR039" H 9750 4450 30  0001 C CNN
+F 0 "#PWR038" H 9750 4450 30  0001 C CNN
 F 1 "GND" H 9750 4380 30  0001 C CNN
 F 2 "" H 9750 4450 60  0000 C CNN
@@
 $EndComp
 $Comp
-L GND #PWR040
+L GND #PWR039
 U 1 1 53D5A72D
 P 3650 3500
-F 0 "#PWR040" H 3650 3500 30  0001 C CNN
+F 0 "#PWR039" H 3650 3500 30  0001 C CNN
 F 1 "GND" H 3650 3430 30  0001 C CNN
 F 2 "" H 3650 3500 60  0000 C CNN
@@
 Wire Wire Line
 	9100 4200 8700 4200
+Wire Wire Line
+	9900 4200 9750 4200
 $EndSCHEMATC
